File: 2040-keypad/2040-keypad.kicad_sch (KiCad schematic)
At the start: 0 parts

Commit message: 2040
Parts:
- added MX1, MX2: MX-NoLED, symbol MX_Alps_Hybrid:MX-NoLED
- added R1, R2: 220R, Resistor_SMD:R_0201_0603Metric, symbol Device:R_Small
- added R3, R4: 5k1, Resistor_SMD:R_0201_0603Metric, symbol Device:R_Small
- added SW1: SW_Push, symbol Switch:SW_Push
- added U1: Pico, RPi_Pico:RPi_Pico_SMD_TH, symbol MCU_RaspberryPi_and_Boards:Pico
- added USB1: HRO-TYPE-C-31-M-12, symbol Type-C:HRO-TYPE-C-31-M-12
Connections:
- new net: R4.1, USB1.10 (CC2)
- new net: R3.2, USB1.4 (CC1)
- new net: U1.TP2, USB1.5 (DN2), USB1.7 (DN1)
- new net: U1.TP3, USB1.6 (DP1), USB1.8 (DP2)
- new net: MX1.2 (ROW), R1.1
- new net: MX2.2 (ROW), R2.1
- new net: SW1.2, U1.32 (GPIO27_ADC1)
- new net +5V: USB1.11 (VBUS), USB1.2 (VBUS)
- new net COL0: MX1.1 (COL), U1.11 (GPIO8)
- new net COL1: MX2.1 (COL), U1.12 (GPIO9)
- new net GND: R3.1, R4.2, SW1.1, U1.23 (GND), U1.TP1, USB1.1 (GND), USB1.12 (GND)
- new net ROW0: R1.2, R2.2, U1.10 (GPIO7)
Other:
- company: (none) -> GroeneDino.nl
- title: (none) -> rp2040 keypad
